Commit message: Robot moving
Adding a test world, where the movement of the robot can be tested.

File: urdf/nav_bot.urdf (robot description, URDF)
Before this commit: robot mogi_bot, 6 links, 5 joints
Links:
- added link camera_link, mass 0.1; collision box size=.03 .03 .03; visual box size=.03 .03 .03
- added link camera_link_optical
Joints:
- added joint camera_joint: type fixed, parent base_link, child camera_link, origin xyz=0.225 0 0.165 rpy=0 0 0, axis 0 1 0
- added joint camera_optical_joint: type fixed, parent camera_link, child camera_link_optical, origin xyz=0 0 0 rpy=-1.5707 0 -1.5707

Commit message: camera relocation

File: urdf/nav_bot.urdf (robot description, URDF)
Before this commit: robot nav_bot, 9 links, 8 joints
Joints:
- joint camera_joint: origin xyz=0.225 0 0.165 rpy=0 0 0 -> xyz=0.35 0 0 rpy=0 0 0

Commit message: add lidar sensor
add lidar, and reduce the size of the collada meshes to gain the speed of the simulation

File: urdf/nav_bot.urdf (robot description, URDF)
Before this commit: robot nav_bot, 9 links, 8 joints
Links:
- added link scan_link, mass 1e-5; collision box size=.07 .07 .07; visual mesh filename=package://navi_stack_hw/meshes/lidar.dae
Joints:
- added joint scan_joint: type fixed, parent base_link, child scan_link, origin xyz=0.225 0 0.185 rpy=0 0 0, axis 0 1 0
